Commit message: Add camera-guided docking perception and recovery

File: src/companion_robot_description/urdf/companion_robot.urdf.xacro (robot description, xacro)
@@ -444,4 +444,34 @@
     material_name="accent_cyan"
     rgba_value="0.00 0.78 0.95 1.0"/>
+  <!-- Rear camera watches the docking marker while the robot reverses. -->
+  <link name="rear_camera_link">
+    <visual name="rear_camera_housing">
+      <geometry>
+        <box size="0.055 0.075 0.045"/>
+      </geometry>
+      <xacro:apply_material material_name="sensor_dark" rgba_value="0.08 0.10 0.13 1.0"/>
+    </visual>
+  </link>
+  <joint name="rear_camera_joint" type="fixed">
+    <parent link="base_link"/>
+    <child link="rear_camera_link"/>
+    <origin xyz="-0.040 0 0.330" rpy="0 0 ${pi}"/>
+  </joint>
+  <xacro:fixed_cylinder_visual
+    name="rear_camera_lens"
+    parent="rear_camera_link"
+    xyz="0.033 0 0"
+    rpy="0 ${pi / 2.0} 0"
+    radius="0.014"
+    length="0.012"
+    material_name="lens_glass"
+    rgba_value="0.01 0.12 0.18 1.0"/>
+  <!-- ROS optical convention: +Z forward, +X right, +Y down. -->
+  <link name="rear_camera_optical_frame"/>
+  <joint name="rear_camera_optical_joint" type="fixed">
+    <parent link="rear_camera_link"/>
+    <child link="rear_camera_optical_frame"/>
+    <origin xyz="0.033 0 0" rpy="${-pi / 2.0} 0 ${-pi / 2.0}"/>
+  </joint>
   <!-- IMU frame is centered inside the chassis and intentionally has no geometry. -->
   <link name="imu_link"/>
@@ -480,4 +510,31 @@
         </noise>
       </lidar>
+    </sensor>
+  </gazebo>
+  <gazebo reference="rear_camera_link">
+    <sensor name="rear_docking_camera" type="camera">
+      <pose>0.033 0 0 0 0 0</pose>
+      <topic>/rear_camera</topic>
+      <gz_frame_id>rear_camera_optical_frame</gz_frame_id>
+      <update_rate>15</update_rate>
+      <always_on>true</always_on>
+      <visualize>false</visualize>
+      <camera>
+        <horizontal_fov>1.3962634</horizontal_fov>
+        <image>
+          <width>640</width>
+          <height>480</height>
+          <format>R8G8B8</format>
+        </image>
+        <clip>
+          <near>0.04</near>
+          <far>5.0</far>
+        </clip>
+        <noise>
+          <type>gaussian</type>
+          <mean>0.0</mean>
+          <stddev>0.002</stddev>
+        </noise>
+      </camera>
     </sensor>
   </gazebo>

Commit message: Add person detection and safe human following behavior

File: src/companion_robot_description/urdf/companion_robot.urdf.xacro (robot description, xacro)
@@ -444,4 +444,11 @@
     material_name="accent_cyan"
     rgba_value="0.00 0.78 0.95 1.0"/>
+  <!-- ROS optical convention: +Z forward, +X right, +Y down. -->
+  <link name="front_camera_optical_frame"/>
+  <joint name="front_camera_optical_joint" type="fixed">
+    <parent link="camera_link"/>
+    <child link="front_camera_optical_frame"/>
+    <origin xyz="0.041 0 0" rpy="${-pi / 2.0} 0 ${-pi / 2.0}"/>
+  </joint>
   <!-- Rear camera watches the docking marker while the robot reverses. -->
   <link name="rear_camera_link">
@@ -512,4 +519,32 @@
         </noise>
       </lidar>
+    </sensor>
+  </gazebo>
+  <!-- Forward RGB stream for simulated person detection and tracking. -->
+  <gazebo reference="camera_link">
+    <sensor name="front_person_camera" type="camera">
+      <pose>0.041 0 0 0 0 0</pose>
+      <topic>/front_camera</topic>
+      <gz_frame_id>front_camera_optical_frame</gz_frame_id>
+      <update_rate>10</update_rate>
+      <always_on>true</always_on>
+      <visualize>false</visualize>
+      <camera>
+        <horizontal_fov>1.3962634</horizontal_fov>
+        <image>
+          <width>424</width>
+          <height>240</height>
+          <format>R8G8B8</format>
+        </image>
+        <clip>
+          <near>0.05</near>
+          <far>6.0</far>
+        </clip>
+        <noise>
+          <type>gaussian</type>
+          <mean>0.0</mean>
+          <stddev>0.004</stddev>
+        </noise>
+      </camera>
     </sensor>
   </gazebo>

Commit message: Add person identity tracking and stabilize human following

File: src/companion_robot_description/urdf/companion_robot.urdf.xacro (robot description, xacro)
@@ -11,4 +11,6 @@
   <xacro:property name="wheel_mass" value="0.35"/>
   <xacro:property name="caster_radius" value="0.025"/>
+  <!-- Keep the 360-degree LiDAR above every other sensor and body part. -->
+  <xacro:property name="lidar_mount_z" value="0.380"/>
   <material name="body_orange">
     <color rgba="0.95 0.32 0.05 1.0"/>
@@ -337,8 +339,22 @@
     </inertial>
   </link>
+  <!--
+    The LiDAR used to sit at z=0.165 m, where its scan plane intersected the
+    forward camera mast. Mount it above both cameras so a 360-degree scan
+    cannot report the robot itself as an obstacle.
+  -->
+  <xacro:fixed_cylinder_visual
+    name="lidar_pedestal"
+    parent="base_link"
+    xyz="-0.045 0 0.269"
+    rpy="0 0 0"
+    radius="0.014"
+    length="0.222"
+    material_name="hub_metal"
+    rgba_value="0.52 0.57 0.64 1.0"/>
   <joint name="lidar_joint" type="fixed">
     <parent link="base_link"/>
     <child link="lidar_link"/>
-    <origin xyz="-0.045 0 ${base_height + 0.045}"/>
+    <origin xyz="-0.045 0 ${lidar_mount_z}"/>
   </joint>
   <xacro:fixed_cylinder_visual
@@ -527,5 +543,5 @@
       <topic>/front_camera</topic>
       <gz_frame_id>front_camera_optical_frame</gz_frame_id>
-      <update_rate>10</update_rate>
+      <update_rate>8</update_rate>
       <always_on>true</always_on>
       <visualize>false</visualize>
@@ -554,5 +570,5 @@
       <topic>/rear_camera</topic>
       <gz_frame_id>rear_camera_optical_frame</gz_frame_id>
-      <update_rate>15</update_rate>
+      <update_rate>10</update_rate>
       <always_on>true</always_on>
       <visualize>false</visualize>
